Commit message: Worked on Fixing Parts Floating in Space Issue

File: irb120.xacro (robot description, xacro)
@@ -273,5 +273,5 @@
     </inertial>
   </link>
-  <link name="mountingConnection">
+<!--  <link name="mountingConnection">
     <collision>
       <origin xyz="0 0 0" rpy="0 0 0"/>
@@ -284,5 +284,5 @@
       <geometry> -->
 	<!--box size="${width} ${width} ${height2}"/-->
-	<mesh filename="package://abb_common/meshes/irb120/visual/mountingConnection.stl" scale="0.001 0.001 0.001"/>
+<!--	<mesh filename="package://abb_common/meshes/irb120/visual/mountingConnection.stl" scale="0.001 0.001 0.001"/>
       </geometry>
       <material name="red"/>
@@ -296,5 +296,5 @@
 	  izz="1.0"/>
     </inertial>
-  </link>
+  </link> -->
   <link name="upperMount">
     <collision>
@@ -345,13 +345,13 @@
     </inertial>
   </link>
-  <joint name="firstEffector" type="continuous">
+  <joint name="firstEffector" type="fixed">
     <parent link="link7"/>
     <child link="bottomMount"/>
-    <origin rpy="0 0 0" xyz="0.072 0 0"/>
+    <origin rpy="0 1.5 0" xyz="0 0 0"/>
     <axis xyz="1 0 0"/>
      <limit effort="20" lower="-6.98132" upper="6.98132" velocity="7.33038"/>
     <dynamics damping="0.7"/>
   </joint>
-  <joint name="middleConnector" type="continuous">
+ <!-- <joint name="middleConnector" type="fixed">
     <parent link="bottomMount"/>
     <child link="mountingConnection"/>
@@ -360,17 +360,17 @@
      <limit effort="20" lower="-6.98132" upper="6.98132" velocity="7.33038"/>
     <dynamics damping="0.7"/>
-  </joint>
-  <joint name="touchesEnd" type="continuous">
-    <parent link="mountingConnection"/>
+  </joint> -->
+  <joint name="touchesEnd" type="fixed">
+    <parent link="bottomMount"/>
     <child link="upperMount"/>
-    <origin rpy="0 0 0" xyz="0.072 0 0"/>
+    <origin rpy="0 0 0" xyz="0 0 -.02"/>
     <axis xyz="1 0 0"/>
      <limit effort="20" lower="-6.98132" upper="6.98132" velocity="7.33038"/>
     <dynamics damping="0.7"/>
   </joint>
-  <joint name="endEffector" type="continuous">
+  <joint name="endEffector" type="fixed">
     <parent link="upperMount"/>
     <child link="paint_gun"/>
-    <origin rpy="0 0 0" xyz="0.072 0 0"/>
+    <origin rpy="0 -1.5 3.14" xyz="0 0 0"/>
     <axis xyz="1 0 0"/>
      <limit effort="20" lower="-6.98132" upper="6.98132" velocity="7.33038"/>
@@ -437,5 +437,5 @@
     </actuator>
   </transmission>
-  <transmission name="tran7">
+ <!-- <transmission name="tran7">
     <type>transmission_interface/SimpleTransmission</type>
     <joint name="firstEffector">
@@ -476,4 +476,4 @@
       <mechanicalReduction>1</mechanicalReduction>
     </actuator>
-  </transmission>
+  </transmission> -->
 </robot>

Commit message: URDF with LBracket, PaintCloud, and Color

File: irb120.xacro (robot description, xacro)
@@ -334,5 +334,33 @@
 	<mesh filename="package://abb_common/meshes/irb120/visual/288048_CAD_model.stl" scale="0.001 0.001 0.001"/>
       </geometry>
-      <material name="red"/>
+      <material name="gun"/>
+      	<color rgba = "0 0 128 1"/>
+      </material>
+    </visual>
+    <inertial>
+      <origin xyz="0 0 0" rpy="0 0 0"/>
+      <mass value="1"/>
+      <inertia
+	  ixx="1.0" ixy="0.0" ixz="0.0"
+	  iyy="1.0" iyz="0.0"
+	  izz="1.0"/>
+    </inertial>
+  </link>
+  <link name="paintTriangle">
+    <collision>
+      <origin xyz="0 0 0" rpy="0 0 0"/>
+      <geometry>
+	<box size="0.1 0.1 0.1"/>
+      </geometry>
+    </collision>
+    <visual>
+      <origin xyz="0 0 0" rpy="0 0 0"/>
+      <geometry> -->
+	<!--box size="${width} ${width} ${height2}"/-->
+	<mesh filename="package://abb_common/meshes/irb120/visual/paintTriangle.stl" scale="0.001 0.001 0.001"/>
+      </geometry>
+      <material name="paint"/>
+      	<color rgba = "255 0 0 1"/>
+      </material>
     </visual>
     <inertial>
@@ -377,4 +405,12 @@
     <dynamics damping="0.7"/>
   </joint>
+  <joint name="paintCloud" type="fixed">
+    <parent link="paint_gun"/>
+    <child link="paintTriangle"/>
+    <origin rpy="0 -1.5 3.14" xyz="0 0 0"/>
+    <axis xyz="1 0 0"/>
+     <limit effort="20" lower="-6.98132" upper="6.98132" velocity="7.33038"/>
+    <dynamics damping="0.7"/>
+  </joint>
   <transmission name="tran1">
     <type>transmission_interface/SimpleTransmission</type>

Commit message: Have all proper components in URDF now and compiles without error

File: irb120.xacro (robot description, xacro)
@@ -10,5 +10,5 @@
   #<xacro:property name="camera_link" value="0.05" /> <!-- Size of square 'camera' box -->
   #<xacro:property name="axel_offset" value="0.05" /> <!-- Space btw top of beam and the each joint -->
-  <!-- Import all Gazebo-customization elements, including Gazebo colors -->
+  <!-- Import all Gazebo-customization elements, including Gazebos -->
   <xacro:include filename="$(find abby_description)/urdf/irb120.gazebo" />
   <!-- Import Rviz colors -->
@@ -22,24 +22,7 @@
   <!-- Base Link -->
   <link name="link1">
-    <!--collision>
-      <origin xyz="0 0 0" rpy="0 0 0"/>
-      <geometry>
-	<box size="0.1 0.1 0.1"/>
-      </geometry>
-    </collision-->
-    <!--visual>
-      <origin xyz="0 0 0" rpy="0 0 0"/>
-      <geometry>
-        <mesh filename="package://abb_common/meshes/irb120/visual/base_link.stl"/>
-      </geometry>
-      <material name="abb_orange">
-        <color rgba="1 0.43 0 1"/>
-      </material>
-    </visua-->
-    <visual>
-      <!--origin xyz="0 0 ${height1/2}" rpy="0 0 0"/-->
+    <visual>
        <origin xyz="0 0 0" rpy="0 0 0"/>
       <geometry>
-	<!--box size="${width} ${width} ${height1}"/-->
 	       <mesh filename="package://abb_common/meshes/irb120/visual/base_link.stl"/>
       </geometry>
@@ -65,14 +48,7 @@
   <!-- Middle Link -->
   <link name="link2">
-    <!--collision>
-      <origin xyz="0 0 0" rpy="0 0 0"/>
-      <geometry>
-	<box size="0.1 0.1 0.1"/>
-      </geometry>
-    </collision-->
-    <visual>
-      <origin xyz="0 0 0" rpy="0 0 0"/>
-      <geometry>
-	<!--box size="${width} ${width} ${height2}"/-->
+    <visual>
+      <origin xyz="0 0 0" rpy="0 0 0"/>
+      <geometry>
 	<mesh filename="package://abb_common/meshes/irb120/collision/link_1.stl"/>
       </geometry>
@@ -258,109 +234,97 @@
     <visual>
       <origin xyz="0 0 0" rpy="0 0 0"/>
-      <geometry> -->
-	<!--box size="${width} ${width} ${height2}"/-->
+      <geometry>
 	<mesh filename="package://abb_common/meshes/irb120/visual/bottomMount.stl" scale="0.001 0.001 0.001"/>
       </geometry>
+    </visual>
+    <inertial>
+      <origin xyz="0 0 0" rpy="0 0 0"/>
+      <mass value="1"/>
+      <inertia
+	  ixx="1.0" ixy="0.0" ixz="0.0"
+	  iyy="1.0" iyz="0.0"
+	  izz="1.0"/>
+    </inertial>
+  </link>
+  <link name="LBracket">
+    <collision>
+      <origin xyz="0 0 0" rpy="0 0 0"/>
+      <geometry>
+	<box size="0.1 0.1 0.1"/>
+      </geometry>
+    </collision>
+    <visual>
+      <origin xyz="0 0 0" rpy="0 0 0"/>
+      <geometry>
+	<mesh filename="package://abb_common/meshes/irb120/visual/LBracket.stl" scale="0.001 0.001 0.001"/>
+      </geometry>
+    </visual>
+    <inertial>
+      <origin xyz="0 0 0" rpy="0 0 0"/>
+      <mass value="1"/>
+      <inertia
+	  ixx="1.0" ixy="0.0" ixz="0.0"
+	  iyy="1.0" iyz="0.0"
+	  izz="1.0"/>
+    </inertial>
+  </link>
+ <link name="upperMount">
+    <collision>
+      <origin xyz="0 0 0" rpy="0 0 0"/>
+      <geometry>
+	<box size="0.1 0.1 0.1"/>
+      </geometry>
+    </collision>
+    <visual>
+      <origin xyz="0 0 0" rpy="0 0 0"/>
+      <geometry>
+	<mesh filename="package://abb_common/meshes/irb120/visual/upperMount.stl" scale="0.001 0.001 0.001"/>
+      </geometry>
+    </visual>
+    <inertial>
+      <origin xyz="0 0 0" rpy="0 0 0"/>
+      <mass value="1"/>
+      <inertia
+	  ixx="1.0" ixy="0.0" ixz="0.0"
+	  iyy="1.0" iyz="0.0"
+	  izz="1.0"/>
+    </inertial>
+  </link>
+  <link name="paint_gun">
+    <collision>
+      <origin xyz="0 0 0" rpy="0 0 0"/>
+      <geometry>
+	<box size="0.1 0.1 0.1"/>
+      </geometry>
+    </collision>
+    <visual>
+      <origin xyz="0 0 0" rpy="0 0 0"/>
+      <geometry>
+	<mesh filename="package://abb_common/meshes/irb120/visual/288048_CAD_model.stl" scale="0.001 0.001 0.001"/>
+      </geometry>
+     <material name="blue"/>
+    </visual>
+    <inertial>
+      <origin xyz="0 0 0" rpy="0 0 0"/>
+      <mass value="1"/>
+      <inertia
+	  ixx="1.0" ixy="0.0" ixz="0.0"
+	  iyy="1.0" iyz="0.0"
+	  izz="1.0"/>
+    </inertial>
+  </link>
+  <link name="paintTriangle">
+    <collision>
+      <origin xyz="0 0 0" rpy="0 0 0"/>
+      <geometry>
+	<box size="0.1 0.1 0.1"/>
+      </geometry>
+    </collision>
+    <visual>
+      <origin xyz="0 0 0" rpy="0 0 0"/>
+      <geometry>
+	<mesh filename="package://abb_common/meshes/irb120/visual/paintTriangle.stl" scale="0.001 0.001 0.001"/>
+      </geometry>
       <material name="red"/>
-    </visual>
-    <inertial>
-      <origin xyz="0 0 0" rpy="0 0 0"/>
-      <mass value="1"/>
-      <inertia
-	  ixx="1.0" ixy="0.0" ixz="0.0"
-	  iyy="1.0" iyz="0.0"
-	  izz="1.0"/>
-    </inertial>
-  </link>
-<!--  <link name="mountingConnection">
-    <collision>
-      <origin xyz="0 0 0" rpy="0 0 0"/>
-      <geometry>
-	<box size="0.1 0.1 0.1"/>
-      </geometry>
-    </collision>
-    <visual>
-      <origin xyz="0 0 0" rpy="0 0 0"/>
-      <geometry> -->
-	<!--box size="${width} ${width} ${height2}"/-->
-<!--	<mesh filename="package://abb_common/meshes/irb120/visual/mountingConnection.stl" scale="0.001 0.001 0.001"/>
-      </geometry>
-      <material name="red"/>
-    </visual>
-    <inertial>
-      <origin xyz="0 0 0" rpy="0 0 0"/>
-      <mass value="1"/>
-      <inertia
-	  ixx="1.0" ixy="0.0" ixz="0.0"
-	  iyy="1.0" iyz="0.0"
-	  izz="1.0"/>
-    </inertial>
-  </link> -->
-  <link name="upperMount">
-    <collision>
-      <origin xyz="0 0 0" rpy="0 0 0"/>
-      <geometry>
-	<box size="0.1 0.1 0.1"/>
-      </geometry>
-    </collision>
-    <visual>
-      <origin xyz="0 0 0" rpy="0 0 0"/>
-      <geometry> -->
-	<!--box size="${width} ${width} ${height2}"/-->
-	<mesh filename="package://abb_common/meshes/irb120/visual/upperMount.stl" scale="0.001 0.001 0.001"/>
-      </geometry>
-      <material name="red"/>
-    </visual>
-    <inertial>
-      <origin xyz="0 0 0" rpy="0 0 0"/>
-      <mass value="1"/>
-      <inertia
-	  ixx="1.0" ixy="0.0" ixz="0.0"
-	  iyy="1.0" iyz="0.0"
-	  izz="1.0"/>
-    </inertial>
-  </link>
-  <link name="paint_gun">
-    <collision>
-      <origin xyz="0 0 0" rpy="0 0 0"/>
-      <geometry>
-	<box size="0.1 0.1 0.1"/>
-      </geometry>
-    </collision>
-    <visual>
-      <origin xyz="0 0 0" rpy="0 0 0"/>
-      <geometry> -->
-	<!--box size="${width} ${width} ${height2}"/-->
-	<mesh filename="package://abb_common/meshes/irb120/visual/288048_CAD_model.stl" scale="0.001 0.001 0.001"/>
-      </geometry>
-      <material name="gun"/>
-      	<color rgba = "0 0 128 1"/>
-      </material>
-    </visual>
-    <inertial>
-      <origin xyz="0 0 0" rpy="0 0 0"/>
-      <mass value="1"/>
-      <inertia
-	  ixx="1.0" ixy="0.0" ixz="0.0"
-	  iyy="1.0" iyz="0.0"
-	  izz="1.0"/>
-    </inertial>
-  </link>
-  <link name="paintTriangle">
-    <collision>
-      <origin xyz="0 0 0" rpy="0 0 0"/>
-      <geometry>
-	<box size="0.1 0.1 0.1"/>
-      </geometry>
-    </collision>
-    <visual>
-      <origin xyz="0 0 0" rpy="0 0 0"/>
-      <geometry> -->
-	<!--box size="${width} ${width} ${height2}"/-->
-	<mesh filename="package://abb_common/meshes/irb120/visual/paintTriangle.stl" scale="0.001 0.001 0.001"/>
-      </geometry>
-      <material name="paint"/>
-      	<color rgba = "255 0 0 1"/>
-      </material>
     </visual>
     <inertial>
@@ -381,14 +345,14 @@
     <dynamics damping="0.7"/>
   </joint>
- <!-- <joint name="middleConnector" type="fixed">
+  <joint name="middle" type="fixed">
     <parent link="bottomMount"/>
-    <child link="mountingConnection"/>
-    <origin rpy="0 0 0" xyz="0.072 0 0"/>
-    <axis xyz="1 0 0"/>
-     <limit effort="20" lower="-6.98132" upper="6.98132" velocity="7.33038"/>
-    <dynamics damping="0.7"/>
-  </joint> -->
+    <child link="LBracket"/>
+    <origin rpy="0 0 0" xyz="0 0 -.02"/>
+    <axis xyz="1 0 0"/>
+     <limit effort="20" lower="-6.98132" upper="6.98132" velocity="7.33038"/>
+    <dynamics damping="0.7"/>
+  </joint>
   <joint name="touchesEnd" type="fixed">
-    <parent link="bottomMount"/>
+    <parent link="LBracket"/>
     <child link="upperMount"/>
     <origin rpy="0 0 0" xyz="0 0 -.02"/>
@@ -473,43 +437,3 @@
     </actuator>
   </transmission>
- <!-- <transmission name="tran7">
-    <type>transmission_interface/SimpleTransmission</type>
-    <joint name="firstEffector">
-      <hardwareInterface>EffortJointInterface</hardwareInterface>
-    </joint>
-    <actuator name="motor7">
-      <hardwareInterface>EffortJointInterface</hardwareInterface>
-      <mechanicalReduction>1</mechanicalReduction>
-    </actuator>
-  </transmission>
-  <transmission name="tran8">
-    <type>transmission_interface/SimpleTransmission</type>
-    <joint name="middleConnector">
-      <hardwareInterface>EffortJointInterface</hardwareInterface>
-    </joint>
-    <actuator name="motor8">
-      <hardwareInterface>EffortJointInterface</hardwareInterface>
-      <mechanicalReduction>1</mechanicalReduction>
-    </actuator>
-  </transmission>
-  <transmission name="tran9">
-    <type>transmission_interface/SimpleTransmission</type>
-    <joint name="touchesEnd">
-      <hardwareInterface>EffortJointInterface</hardwareInterface>
-    </joint>
-    <actuator name="motor9">
-      <hardwareInterface>EffortJointInterface</hardwareInterface>
-      <mechanicalReduction>1</mechanicalReduction>
-    </actuator>
-  </transmission>
-  <transmission name="tran10">
-    <type>transmission_interface/SimpleTransmission</type>
-    <joint name="endEffector">
-      <hardwareInterface>EffortJointInterface</hardwareInterface>
-    </joint>
-    <actuator name="motor10">
-      <hardwareInterface>EffortJointInterface</hardwareInterface>
-      <mechanicalReduction>1</mechanicalReduction>
-    </actuator>
-  </transmission> -->
 </robot>

Commit message: URDF stl parts now have color

File: irb120.xacro (robot description, xacro)
@@ -206,5 +206,5 @@
 	        <mesh filename="package://abb_common/meshes/irb120/visual/link_6.stl"/>
       </geometry>
-      <material name="orange"/>
+      <material name="grey"/>
     </visual>
     <inertial>
@@ -225,5 +225,5 @@
     <dynamics damping="0.7"/>
   </joint>
-  <link name="bottomMount">
+  <link name="LBracket">
     <collision>
       <origin xyz="0 0 0" rpy="0 0 0"/>
@@ -233,19 +233,20 @@
     </collision>
     <visual>
-      <origin xyz="0 0 0" rpy="0 0 0"/>
-      <geometry>
-	<mesh filename="package://abb_common/meshes/irb120/visual/bottomMount.stl" scale="0.001 0.001 0.001"/>
-      </geometry>
-    </visual>
-    <inertial>
-      <origin xyz="0 0 0" rpy="0 0 0"/>
-      <mass value="1"/>
-      <inertia
-	  ixx="1.0" ixy="0.0" ixz="0.0"
-	  iyy="1.0" iyz="0.0"
-	  izz="1.0"/>
-    </inertial>
-  </link>
-  <link name="LBracket">
+      <origin xyz="0 0 0" rpy="1.57 0 0"/>
+      <geometry>
+	<mesh filename="package://abb_common/meshes/irb120/visual/LBracket.stl" scale="0.001 0.001 0.001"/>
+      </geometry>
+	<material name="white"/>
+    </visual>
+    <inertial>
+      <origin xyz="0 0 0" rpy="0 0 0"/>
+      <mass value="1"/>
+      <inertia
+	  ixx="1.0" ixy="0.0" ixz="0.0"
+	  iyy="1.0" iyz="0.0"
+	  izz="1.0"/>
+    </inertial>
+  </link>
+  <link name="paint_gun">
     <collision>
       <origin xyz="0 0 0" rpy="0 0 0"/>
@@ -255,19 +256,20 @@
     </collision>
     <visual>
-      <origin xyz="0 0 0" rpy="0 0 0"/>
-      <geometry>
-	<mesh filename="package://abb_common/meshes/irb120/visual/LBracket.stl" scale="0.001 0.001 0.001"/>
-      </geometry>
-    </visual>
-    <inertial>
-      <origin xyz="0 0 0" rpy="0 0 0"/>
-      <mass value="1"/>
-      <inertia
-	  ixx="1.0" ixy="0.0" ixz="0.0"
-	  iyy="1.0" iyz="0.0"
-	  izz="1.0"/>
-    </inertial>
-  </link>
- <link name="upperMount">
+      <origin xyz="0.02 -0.025 0.0525" rpy="1.57 1.5 0"/>
+      <geometry>
+	<mesh filename="package://abb_common/meshes/irb120/visual/288048_CAD_model.stl" scale="0.001 0.001 0.001"/>
+      </geometry>
+     <material name="blue"/>
+    </visual>
+    <inertial>
+      <origin xyz="0 0 0" rpy="0 0 0"/>
+      <mass value="1"/>
+      <inertia
+	  ixx="1.0" ixy="0.0" ixz="0.0"
+	  iyy="1.0" iyz="0.0"
+	  izz="1.0"/>
+    </inertial>
+  </link>
+  <link name="paintTriangle">
     <collision>
       <origin xyz="0 0 0" rpy="0 0 0"/>
@@ -277,50 +279,5 @@
     </collision>
     <visual>
-      <origin xyz="0 0 0" rpy="0 0 0"/>
-      <geometry>
-	<mesh filename="package://abb_common/meshes/irb120/visual/upperMount.stl" scale="0.001 0.001 0.001"/>
-      </geometry>
-    </visual>
-    <inertial>
-      <origin xyz="0 0 0" rpy="0 0 0"/>
-      <mass value="1"/>
-      <inertia
-	  ixx="1.0" ixy="0.0" ixz="0.0"
-	  iyy="1.0" iyz="0.0"
-	  izz="1.0"/>
-    </inertial>
-  </link>
-  <link name="paint_gun">
-    <collision>
-      <origin xyz="0 0 0" rpy="0 0 0"/>
-      <geometry>
-	<box size="0.1 0.1 0.1"/>
-      </geometry>
-    </collision>
-    <visual>
-      <origin xyz="0 0 0" rpy="0 0 0"/>
-      <geometry>
-	<mesh filename="package://abb_common/meshes/irb120/visual/288048_CAD_model.stl" scale="0.001 0.001 0.001"/>
-      </geometry>
-     <material name="blue"/>
-    </visual>
-    <inertial>
-      <origin xyz="0 0 0" rpy="0 0 0"/>
-      <mass value="1"/>
-      <inertia
-	  ixx="1.0" ixy="0.0" ixz="0.0"
-	  iyy="1.0" iyz="0.0"
-	  izz="1.0"/>
-    </inertial>
-  </link>
-  <link name="paintTriangle">
-    <collision>
-      <origin xyz="0 0 0" rpy="0 0 0"/>
-      <geometry>
-	<box size="0.1 0.1 0.1"/>
-      </geometry>
-    </collision>
-    <visual>
-      <origin xyz="0 0 0" rpy="0 0 0"/>
+      <origin xyz="0 0 0" rpy="-3.14 0 0"/>
       <geometry>
 	<mesh filename="package://abb_common/meshes/irb120/visual/paintTriangle.stl" scale="0.001 0.001 0.001"/>
@@ -337,7 +294,7 @@
     </inertial>
   </link>
-  <joint name="firstEffector" type="fixed">
+  <joint name="firstEffector" type="continuous">
     <parent link="link7"/>
-    <child link="bottomMount"/>
+    <child link="LBracket"/>
     <origin rpy="0 1.5 0" xyz="0 0 0"/>
     <axis xyz="1 0 0"/>
@@ -345,7 +302,7 @@
     <dynamics damping="0.7"/>
   </joint>
-  <joint name="middle" type="fixed">
-    <parent link="bottomMount"/>
-    <child link="LBracket"/>
+  <joint name="touchesEnd" type="continuous">
+    <parent link="LBracket"/>
+    <child link="paint_gun"/>
     <origin rpy="0 0 0" xyz="0 0 -.02"/>
     <axis xyz="1 0 0"/>
@@ -353,21 +310,5 @@
     <dynamics damping="0.7"/>
   </joint>
-  <joint name="touchesEnd" type="fixed">
-    <parent link="LBracket"/>
-    <child link="upperMount"/>
-    <origin rpy="0 0 0" xyz="0 0 -.02"/>
-    <axis xyz="1 0 0"/>
-     <limit effort="20" lower="-6.98132" upper="6.98132" velocity="7.33038"/>
-    <dynamics damping="0.7"/>
-  </joint>
-  <joint name="endEffector" type="fixed">
-    <parent link="upperMount"/>
-    <child link="paint_gun"/>
-    <origin rpy="0 -1.5 3.14" xyz="0 0 0"/>
-    <axis xyz="1 0 0"/>
-     <limit effort="20" lower="-6.98132" upper="6.98132" velocity="7.33038"/>
-    <dynamics damping="0.7"/>
-  </joint>
-  <joint name="paintCloud" type="fixed">
+  <joint name="paintCloud" type="continuous">
     <parent link="paint_gun"/>
     <child link="paintTriangle"/>
